Commit message: Rebase from 'debian/noetic/tesseract_support'

File: urdf/abb_irb2400.urdf (robot description, URDF)
Before this commit: robot abb_irb2400, 9 links, 8 joints
Links:
- link base_link: geometry collision mesh filename=package://tesseract_support/meshes/abb_irb2400/irb2400/coll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; visual mesh filename=package://tesseract_support/meshes/abb_irb2400/irb2400/visu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
- link link_1: geometry collision mesh filename=package://tesseract_support/meshes/abb_irb2400/irb2400/coll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; visual mesh filename=package://tesseract_support/meshes/abb_irb2400/irb2400/visu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
- link link_2: geometry collision mesh filename=package://tesseract_support/meshes/abb_irb2400/irb2400/coll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; visual mesh filename=package://tesseract_support/meshes/abb_irb2400/irb2400/visu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
- link link_3: geometry collision mesh filename=package://tesseract_support/meshes/abb_irb2400/irb2400/coll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; visual mesh filename=package://tesseract_support/meshes/abb_irb2400/irb2400/visu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
- link link_4: geometry collision mesh filename=package://tesseract_support/meshes/abb_irb2400/irb2400/coll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; visual mesh filename=package://tesseract_support/meshes/abb_irb2400/irb2400/visu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
- link link_5: geometry collision mesh filename=package://tesseract_support/meshes/abb_irb2400/irb2400/coll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; visual mesh filename=package://tesseract_support/meshes/abb_irb2400/irb2400/visu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
- link link_6: geometry collision mesh filename=package://tesseract_support/meshes/abb_irb2400/irb2400/coll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; visual mesh filename=package://tesseract_support/meshes/abb_irb2400/irb2400/visu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

File: urdf/abb_irb2400_external_positioner.urdf (robot description, URDF)
Before this commit: robot abb_irb2400_external_positioner, 13 links, 12 joints
Links:
- link base_link: geometry collision mesh filename=package://tesseract_support/meshes/abb_irb2400/irb2400/coll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; visual mesh filename=package://tesseract_support/meshes/abb_irb2400/irb2400/visu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
- link link_1: geometry collision mesh filename=package://tesseract_support/meshes/abb_irb2400/irb2400/coll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; visual mesh filename=package://tesseract_support/meshes/abb_irb2400/irb2400/visu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
- link link_2: geometry collision mesh filename=package://tesseract_support/meshes/abb_irb2400/irb2400/coll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; visual mesh filename=package://tesseract_support/meshes/abb_irb2400/irb2400/visu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
- link link_3: geometry collision mesh filename=package://tesseract_support/meshes/abb_irb2400/irb2400/coll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; visual mesh filename=package://tesseract_support/meshes/abb_irb2400/irb2400/visu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
- link link_4: geometry collision mesh filename=package://tesseract_support/meshes/abb_irb2400/irb2400/coll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; visual mesh filename=package://tesseract_support/meshes/abb_irb2400/irb2400/visu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
- link link_5: geometry collision mesh filename=package://tesseract_support/meshes/abb_irb2400/irb2400/coll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; visual mesh filename=package://tesseract_support/meshes/abb_irb2400/irb2400/visu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
- link link_6: geometry collision mesh filename=package://tesseract_support/meshes/abb_irb2400/irb2400/coll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; visual mesh filename=package://tesseract_support/meshes/abb_irb2400/irb2400/visu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

File: urdf/abb_irb2400_on_positioner.urdf (robot description, URDF)
Before this commit: robot abb_irb2400_on_positioner, 11 links, 10 joints
Links:
- link base_link: geometry collision mesh filename=package://tesseract_support/meshes/abb_irb2400/irb2400/coll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; visual mesh filename=package://tesseract_support/meshes/abb_irb2400/irb2400/visu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
- link link_1: geometry collision mesh filename=package://tesseract_support/meshes/abb_irb2400/irb2400/coll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; visual mesh filename=package://tesseract_support/meshes/abb_irb2400/irb2400/visu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
- link link_2: geometry collision mesh filename=package://tesseract_support/meshes/abb_irb2400/irb2400/coll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; visual mesh filename=package://tesseract_support/meshes/abb_irb2400/irb2400/visu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
- link link_3: geometry collision mesh filename=package://tesseract_support/meshes/abb_irb2400/irb2400/coll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; visual mesh filename=package://tesseract_support/meshes/abb_irb2400/irb2400/visu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
- link link_4: geometry collision mesh filename=package://tesseract_support/meshes/abb_irb2400/irb2400/coll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; visual mesh filename=package://tesseract_support/meshes/abb_irb2400/irb2400/visu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
- link link_5: geometry collision mesh filename=package://tesseract_support/meshes/abb_irb2400/irb2400/coll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; visual mesh filename=package://tesseract_support/meshes/abb_irb2400/irb2400/visu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
- link link_6: geometry collision mesh filename=package://tesseract_support/meshes/abb_irb2400/irb2400/coll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; visual mesh filename=package://tesseract_support/meshes/abb_irb2400/irb2400/visu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

File: urdf/iiwa7.urdf (robot description, URDF)
Before this commit: robot kuka_liwa_7, 11 links, 10 joints
Links:
- link link_0: geometry collision mesh filename=package://tesseract_support/meshes/iiwa7/collision/link_0.s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; visual mesh filename=package://tesseract_support/meshes/iiwa7/visual/link_0.stl
- link link_1: geometry collision mesh filename=package://tesseract_support/meshes/iiwa7/collision/link_1.s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; visual mesh filename=package://tesseract_support/meshes/iiwa7/visual/link_1.stl
- link link_2: geometry collision mesh filename=package://tesseract_support/meshes/iiwa7/collision/link_2.s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; visual mesh filename=package://tesseract_support/meshes/iiwa7/visual/link_2.stl
- link link_3: geometry collision mesh filename=package://tesseract_support/meshes/iiwa7/collision/link_3.s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; visual mesh filename=package://tesseract_support/meshes/iiwa7/visual/link_3.stl
- link link_4: geometry collision mesh filename=package://tesseract_support/meshes/iiwa7/collision/link_4.s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; visual mesh filename=package://tesseract_support/meshes/iiwa7/visual/link_4.stl
- link link_5: geometry collision mesh filename=package://tesseract_support/meshes/iiwa7/collision/link_5.s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; visual mesh filename=package://tesseract_support/meshes/iiwa7/visual/link_5.stl
- link link_6: geometry collision mesh filename=package://tesseract_support/meshes/iiwa7/collision/link_6.s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; visual mesh filename=package://tesseract_support/meshes/iiwa7/visual/link_6.stl
- link link_7: geometry collision mesh filename=package://tesseract_support/meshes/iiwa7/collision/link_7.s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; visual mesh filename=package://tesseract_support/meshes/iiwa7/visual/link_7.stl

File: urdf/lbr_iiwa_14_r820.urdf (robot description, URDF)
Before this commit: robot kuka_lbr_iiwa_14_r820, 10 links, 9 joints
Links:
- link base_link: geometry collision mesh filename=package://tesseract_support/meshes/lbr_iiwa_14_r820/collisi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; visual mesh filename=package://tesseract_support/meshes/lbr_iiwa_14_r820/visual/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
- link link_1: geometry collision mesh filename=package://tesseract_support/meshes/lbr_iiwa_14_r820/collisi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; visual mesh filename=package://tesseract_support/meshes/lbr_iiwa_14_r820/visual/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
- link link_2: geometry collision mesh filename=package://tesseract_support/meshes/lbr_iiwa_14_r820/collisi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; visual mesh filename=package://tesseract_support/meshes/lbr_iiwa_14_r820/visual/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
- link link_3: geometry collision mesh filename=package://tesseract_support/meshes/lbr_iiwa_14_r820/collisi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; visual mesh filename=package://tesseract_support/meshes/lbr_iiwa_14_r820/visual/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
- link link_4: geometry collision mesh filename=package://tesseract_support/meshes/lbr_iiwa_14_r820/collisi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; visual mesh filename=package://tesseract_support/meshes/lbr_iiwa_14_r820/visual/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
- link link_5: geometry collision mesh filename=package://tesseract_support/meshes/lbr_iiwa_14_r820/collisi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; visual mesh filename=package://tesseract_support/meshes/lbr_iiwa_14_r820/visual/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
- link link_6: geometry collision mesh filename=package://tesseract_support/meshes/lbr_iiwa_14_r820/collisi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; visual mesh filename=package://tesseract_support/meshes/lbr_iiwa_14_r820/visual/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
- link link_7: geometry collision mesh filename=package://tesseract_support/meshes/lbr_iiwa_14_r820/collisi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; visual mesh filename=package://tesseract_support/meshes/lbr_iiwa_14_r820/visual/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
